File: Detector Electronics/DetInterfaceCard/NN22_RPi_DetAdapter02_s00.brd (EAGLE design)
At the start: 63.5 x 33 mm, 238 parts, among them J1 M17X2, J2 M05X2_SMD_0.050_NOCREAM, J3 M03X1_0.050_SMD_NO_CREAM, J4 USB-MICRO, J5 M20X2_HARFLEX_M, U1 AD7380, U10 RP2040, U11 MCP1755_DFN, U12 MCP1755_DFN, U13 ADP7142_WSON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

Commit message: Updating detector interface card and adding gerbers.
Parts:
- moved TP20 0.40 mm to (38.7, 6.99)
Routing:
- net VBUS: track 43.7 -> 40.1 mm
- net OPT_EN_VN: track 53.9 -> 51.4 mm
- net OPT_EN_VP: track 54.7 -> 52.4 mm
- net A_COMM: track 61.6 -> 59.7 mm
- net V9P0: track 49.8 -> 51.6 mm
- net VN22: track 42.0 -> 42.8 mm
- net GND: vias 183 -> 182
Other:
- outline, holes or cut-outs redrawn
- board text added: "NinjaNIRS 2022 Detector Interface v02 12/2023"
- board text removed: "NinjaNIRS 2022 Detector Interface v01 4/2023"
